File: HW/IO256/IO256.kicad_pcb (KiCad board)
At the start: 2 copper layers, 170 x 120 mm, 270 parts, among them J1 Conn_02x04_Odd_Even, J10 Conn_02x04_Counter_Clockwise, J102 USB_B, J103 Conn_01x06, J11 Conn_02x04_Counter_Clockwise, J12 Conn_02x04_Counter_Clockwise, J13 Conn_02x04_Counter_Clockwise, J14 Conn_02x04_Counter_Clockwise, J15 Conn_02x04_Counter_Clockwise, J16 Conn_02x04_Counter_Clockwise, J17 Conn_01x04, J18 Conn_02x03_Odd_Even, J19 Conn_02x03_Odd_Even, J20 Conn_02x03_Odd_Even, J21 Conn_01x04, J22 Conn_02x02_Odd_Even, J23 Conn_02x03_Odd_Even, J24 Conn_01x06, J25 USB_B, J3 Conn_01x06, J4 Conn_02x18_Odd_Even, J5 Conn_02x04_Counter_Clockwise, J6 ATX-24, J7 Conn_02x04_Counter_Clockwise, J8 Conn_02x04_Counter_Clockwise, J9 Conn_02x04_Counter_Clockwise, Q2 AO3400A, SW1 SW_Push_DPDT, SW2 SW_Push_DPDT, SW3 SW_Push_DPDT, SW4 SW_Push_DPDT, SW5 SW_Push_DPDT, SW6 SW_Push_DPDT, SW7 SW_DIP_x04, SW8 SW_Push_DPDT, U1 XC6206P332MR, U2 SP3485, U3 TL084C, U4 TL084C, U5 TL084C, U6 STM32G030C, U7 TL084C, U8 SRV05-4

Commit message: update
Parts:
- SW7: footprint Button_Switch_SMD:SW_DIP_SPSTx04_Slide_Copal_CHS-04B_W7.62mm_P1.27mm -> Button_Switch_THT:SW_DIP_SPSTx04_Slide_9.78x12.34mm_W7.62mm_P2.54mm
- moved SW7 9.23 mm to (102.0, 143.2), turned to -90 degrees
Connections:
- SW7 pad 1: GND -> SET4
- SW7 pad 2: GND -> SET3
- SW7 pad 3: GND -> SET2
- SW7 pad 4: GND -> SET1
- SW7 pad 5: SET4 -> GND
- SW7 pad 6: SET3 -> GND
- SW7 pad 7: SET2 -> GND
- SW7 pad 8: SET1 -> GND
Routing:
- net GND: track 424.3 -> 408.9 mm, vias 514 -> 508
- net SET4: track 36.4 -> 29.4 mm
- net SET3: track 37.2 -> 31.5 mm
- net SET2: track 38.1 -> 33.4 mm
- net SET1: track 39.5 -> 36.1 mm
Other:
- board text added: "V13"
- board text removed: "V12"

Commit message: update
Parts:
- U6: value STM32G030C -> STM32G030C8T6
Other:
- board text added: "INPUT_MUX"
- board text added: "J6"
