File: HW/IO256/IO256.kicad_sch (KiCad schematic)
At the start: 48 parts, among them J1 Conn_02x04_Odd_Even, J10 Conn_02x04_Counter_Clockwise, J101 Conn_02x30_Row_Letter_First, J102 USB_B, J103 Conn_01x06, J11 Conn_02x04_Counter_Clockwise, J12 Conn_02x04_Counter_Clockwise, J13 Conn_02x04_Counter_Clockwise, J14 Conn_02x04_Counter_Clockwise, J15 Conn_02x04_Counter_Clockwise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

Commit message: update
Parts:
- J101, J2: now not fitted
- SW1, SW8: value SW_Push_DPDT -> SW6*6_selflock
- SW2, SW3, SW4, SW5, SW6: value SW_Push_DPDT -> SW6*6_button
- renumbered R5 to R108, R5 to R109, R5 to R110, R5 to R111, R5 to R112, R5 to R113
