File: HW/IO256/OPA.kicad_sch (KiCad schematic)
At the start: 132 parts, among them U4 TL084C, U5 TL084C, U7 TL084C, U8 TL084C

Commit message: update
Other:
- company: (none) -> Analog Dragon
- title: (none) -> System 256 REFUTA
Changed lines of the file:
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@@
 (kicad_sch (version 20230121) (generator eeschema)
   (paper "A4")
+  (title_block
+    (title "System 256 REFUTA")
+    (date "2023-10-27")
+    (rev "V13")
+    (company "Analog Dragon")
+  )
   (junction (at 57.15 81.28) (diameter 0) (color 0 0 0 0)
   )

Commit message: update
Parts:
- renumbered C23 to C1, C35 to C10, C36 to C11, C37 to C12, C38 to C15, C43 to C16, C44 to C21, C45 to C22, C46 to C23, C47 to C24, C48 to C25, C49 to C26, C24 to C3, C50 to C35, C52 to C36, C53 to C37, C54 to C38, C25 to C4, C55 to C43, C56 to C44, C57 to C45, C58 to C46, C59 to C47, C26 to C5, D11 to D10, D12 to D11, D13 to D12, D14 to D13, D16 to D14, D17 to D16, D18 to D17, D19 to D18, D20 to D19, D21 to D20, D22 to D21, D23 to D22, D24 to D23, D25 to D24, D26 to D25, D27 to D26, D28 to D27, D29 to D28, D30 to D29, D31 to D30, D32 to D31, D33 to D32, D34 to D33, D35 to D34, R31 to R1, R104 to R100, R105 to R101, R106 to R102, R107 to R103, R108 to R104, R109 to R105, R110 to R106, R111 to R107, R33 to R13, R34 to R14, R36 to R31, R37 to R32, R38 to R33, R39 to R34, R40 to R36, R41 to R37, R42 to R38, R43 to R39, R44 to R40, R45 to R41, R46 to R42, R47 to R43, R48 to R44, R49 to R45, R50 to R46, R51 to R47, R52 to R48, R53 to R49, R54 to R50, R55 to R51, R56 to R52, R57 to R53, R58 to R54, R59 to R55, R60 to R56, R61 to R57, R62 to R58, R63 to R59, R32 to R6, R64 to R60, R65 to R61, R66 to R62, R67 to R63, R68 to R64, R69 to R65, R70 to R66, R71 to R67, R72 to R68, R73 to R69, R74 to R70, R75 to R71, R76 to R72, R77 to R73, R78 to R74, R79 to R75, R80 to R76, R81 to R77, R82 to R78, R83 to R79, R84 to R80, R85 to R81, R86 to R82, R87 to R83, R88 to R84, R89 to R85, R90 to R86, R91 to R87, R92 to R88, R93 to R89, R94 to R90, R95 to R91, R96 to R92, R97 to R93, R98 to R94, R99 to R95, R100 to R96, R101 to R97, R102 to R98, R103 to R99, U4 to U3, U5 to U4, U7 to U5, U8 to U7
