File: HW/IO256/SIF PCB.kicad_sch (KiCad schematic)
At the start: 92 parts, among them J17 Conn_01x04, J18 Conn_02x03_Odd_Even, J19 Conn_02x03_Odd_Even, J20 Conn_02x03_Odd_Even, J21 Conn_01x04, J23 Conn_02x03_Odd_Even, Q2 AO3400A, SW7 SW_DIP_x04, U1 XC6206P332MR, U2 SP3485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

Commit message: update
Parts:
- SW7: footprint Button_Switch_SMD:SW_DIP_SPSTx04_Slide_Copal_CHS-04B_W7.62mm_P1.27mm -> Button_Switch_THT:SW_DIP_SPSTx04_Slide_9.78x12.34mm_W7.62mm_P2.54mm
Connections:
- net GND: now also SW7.5, SW7.6, SW7.7, SW7.8; no longer SW7.1, SW7.2, SW7.3, SW7.4
- net SET1: now also SW7.4; no longer SW7.8
- net SET2: now also SW7.3; no longer SW7.7
- net SET3: now also SW7.2; no longer SW7.6
- net SET4: now also SW7.1; no longer SW7.5
Other:
- company: (none) -> Analog Dragon
- title: (none) -> System 256 REFUTA
- moved on the sheet: SW7
Changed lines of the file:
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@@
 (kicad_sch (version 20230121) (generator eeschema)
   (paper "A4")
-  (junction (at 36.83 100.33) (diameter 0) (color 0 0 0 0)
+  (title_block
+    (title "System 256 REFUTA")
+    (date "2023-10-27")
+    (rev "V13")
+    (company "Analog Dragon")
   )
-  (junction (at 44.45 165.1) (diameter 0) (color 0 0 0 0)
+  (junction (at 36.83 100.33) (diameter 0) (color 0 0 0 0)
   )
   (junction (at 252.73 142.24) (diameter 0) (color 0 0 0 0)
@@
   (junction (at 160.02 39.37) (diameter 0) (color 0 0 0 0)
   )
-  (junction (at 44.45 167.64) (diameter 0) (color 0 0 0 0)
-  )
   (junction (at 153.67 69.85) (diameter 0) (color 0 0 0 0)
   )
@@
   (junction (at 46.99 54.61) (diameter 0) (color 0 0 0 0)
   )
+  (junction (at 44.45 162.56) (diameter 0) (color 0 0 0 0)
+  )
+  (junction (at 44.45 167.64) (diameter 0) (color 0 0 0 0)
+  )
   (junction (at 88.9 53.34) (diameter 0) (color 0 0 0 0)
   )
@@
   (junction (at 153.67 24.13) (diameter 0) (color 0 0 0 0)
   )
-  (junction (at 44.45 162.56) (diameter 0) (color 0 0 0 0)
+  (junction (at 44.45 165.1) (diameter 0) (color 0 0 0 0)
   )
   (junction (at 82.55 24.13) (diameter 0) (color 0 0 0 0)
@@
     (stroke (width 0) (type default))
   )
+  (wire (pts (xy 44.45 167.64) (xy 44.45 170.18))
+    (stroke (width 0) (type default))
+  )
   (wire (pts (xy 35.56 86.36) (xy 41.91 86.36))
     (stroke (width 0) (type default))
@@
     (stroke (width 0) (type default))
   )
-  (wire (pts (xy 44.45 162.56) (xy 44.45 165.1))
-    (stroke (width 0) (type default))
-  )
   (wire (pts (xy 46.99 71.12) (xy 52.07 71.12))
     (stroke (width 0) (type default))
@@
     (stroke (width 0) (type default))
   )
-  (wire (pts (xy 44.45 167.64) (xy 44.45 170.18))
-    (stroke (width 0) (type default))
-  )
   (wire (pts (xy 50.8 34.29) (xy 54.61 34.29))
     (stroke (width 0) (type default))
@@
     (stroke (width 0) (type default))
   )
+  (wire (pts (xy 44.45 162.56) (xy 44.45 165.1))
+    (stroke (width 0) (type default))
+  )
   (polyline (pts (xy 16.51 180.34) (xy 68.58 180.34))
     (stroke (width 0) (type default))
@@
     (stroke (width 0) (type default))
   )
+  (wire (pts (xy 44.45 165.1) (xy 44.45 167.64))
+    (stroke (width 0) (type default))
+  )
   (wire (pts (xy 52.07 81.28) (xy 52.07 92.71))
     (stroke (width 0) (type default))
@@
     (stroke (width 0) (type default))
   )
-  (wire (pts (xy 44.45 165.1) (xy 44.45 167.64))
-    (stroke (width 0) (type default))
-  )
   (wire (pts (xy 88.9 71.12) (xy 95.25 71.12))
     (stroke (width 0) (type default))
@@
     )
   )
-  (symbol (lib_id "Switch:SW_DIP_x04") (at 52.07 165.1 0) (unit 1)
+  (symbol (lib_id "Switch:SW_DIP_x04") (at 52.07 162.56 180) (unit 1)
     (in_bom yes) (on_board yes) (dnp no)
-    (property "Reference" "SW7" (at 52.07 156.21 0)
+    (property "Reference" "SW7" (at 52.07 171.45 0)
       (effects (font (size 1.27 1.27)))
     )
-    (property "Value" "SW_DIP_x04" (at 52.07 156.3171 0)
+    (property "Value" "SW_DIP_x04" (at 52.07 171.3429 0)
       (effects (font (size 1.27 1.27)) hide)
     )
-    (property "Footprint" "Button_Switch_SMD:SW_DIP_SPSTx04_Slide_Copal_CHS-04B_W7.62mm_P1.27mm" (at 52.07 165.1 0)
+    (property "Footprint" "Button_Switch_THT:SW_DIP_SPSTx04_Slide_9.78x12.34mm_W7.62mm_P2.54mm" (at 52.07 162.56 0)
       (effects (font (size 1.27 1.27)) hide)
     )
-    (property "Datasheet" "~" (at 52.07 165.1 0)
+    (property "Datasheet" "~" (at 52.07 162.56 0)
       (effects (font (size 1.27 1.27)) hide)
     )

Commit message: update
Parts:
- U6: value STM32G030C -> STM32G030C8T6
